Commit message: 0520update

File: resources/robots/h1_2_centaur/h1_2_12dof_centaur_fixed.urdf (robot description, URDF)
Before this commit: robot h1_5, 73 links, 73 joints
Links:
- added link CTimu_link; visual box size=0.02 0.02 0.02
- link imu_link: geometry 
Joints:
- joint torso_imu_joint: child imu_link -> CTimu_link
- joint torso_joint: axis 0 1 0 -> 0 0 1; limit lower=-1.0 upper=0.1 effort=800 velocity=23 -> lower=-2.35 upper=2.35 effort=200 velocity=23; type revolute -> fixed
